File: co2_sensor_module/can.kicad_sch (KiCad schematic)
At the start: 7 parts, among them U8 TJA1042T-3

Commit message: first draft of sensor schematic is done!
Connections:
- net PV50: now reaches C16.1, C17.1, U8.3 (VCC)
Changed lines of the file:
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@@
 		(color 0 0 0 0)
 	)
+	(junction
+		(at 36.83 39.37)
+		(diameter 0)
+		(color 0 0 0 0)
+	)
 	(wire
 		(pts
@@
 	(wire
 		(pts
+			(xy 35.56 39.37) (xy 36.83 39.37)
+		)
+		(stroke
+			(width 0)
+			(type default)
+		)
+	)
+	(wire
+		(pts
 			(xy 97.79 54.61) (xy 109.22 54.61)
 		)
@@
 		)
 	)
+	(hierarchical_label "PV50"
+		(shape input)
+		(at 35.56 39.37 180)
+		(effects
+			(font
+				(size 1.27 1.27)
+			)
+			(justify right)
+		)
+	)
