File: co2_sensor_module/mcu.kicad_sch (KiCad schematic)
At the start: 13 parts, among them J1 Conn_ARM_SWD_TagConnect_TC203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, U1 STM32L431KBUx

Commit message: mostly done w/ sensor module
Parts:
- removed C1, C2: 100nF, symbol Device:C_Small
- removed C5, C6: 1uF, symbol Device:C_Small
- removed R3, R4: 10K, symbol Device:R_Small
- added C18, C21: 1uF, Capacitor_SMD:C_0603_1608Metric, symbol Device:C_Small
- added C19, C20: 100nF, Capacitor_SMD:C_0402_1005Metric, symbol Device:C_Small
- added D2: LED_Red, LED_SMD:LED_0805_2012Metric, symbol Device:LED_Small
- added D3: LED_Green, LED_SMD:LED_0805_2012Metric, symbol Device:LED_Small
- added R12, R13, R14, R15: 100K, symbol Device:R_Small
- added R17, R18, R19, R20: 10K, Resistor_SMD:R_0402_1005Metric, symbol Device:R_Small
- added SW1: SW_DIP_x04, Button_Switch_THT:SW_DIP_SPSTx04_Slide_9.78x12.34mm_W7.62mm_P2.54mm, symbol Switch:SW_DIP_x04
- C3: footprint (none) -> Capacitor_SMD:C_0402_1005Metric; LCSC (none) -> C15195
- C4: footprint (none) -> Capacitor_SMD:C_0603_1608Metric; LCSC (none) -> C19666
- R1, R2: value 10K -> 200; footprint (none) -> Resistor_SMD:R_0603_1608Metric; LCSC (none) -> C8218
- U2: value (none) -> CBLW 24C02
Connections:
- net GND: now also R1.2, R2.2, C18.1, C19.1, C20.1, C21.2, SW1.1, SW1.2, SW1.3, SW1.4
- net I2C_SCL: now also R20.2; no longer R1.2
- net I2C_SDA: now also R19.2; no longer R2.2
- net P3V3: now also C18.2, C19.2, C20.2, C21.1, R12.2, R13.2, R14.2, R15.2, R17.2, R18.2, R19.1, R20.1; no longer R1.1, R2.1
- net at U1.31 (PH3): now also R17.1
- net at U1.6 (PA0), U2.5 (WP): now also R18.1
- net at U1.14 (PB0): now also R15.1, SW1.8
- net at U1.15 (PB1): now also R14.1, SW1.7
- net at U1.21 (PA11): now also D3.2 (A)
- net at U1.22 (PA12): now also D2.2 (A)
- net at U1.26 (PB3): now also R13.1, SW1.6
- net at U1.27 (PB4): now also R12.1, SW1.5
- new net: D2.1 (K), R1.1
- new net: D3.1 (K), R2.1
Other:
- note added: "Sensor Address"

Commit message: first draft of sensor schematic is done!
Parts:
- removed R12, R13, R14, R15: 100K, symbol Device:R_Small
- removed U1: STM32L431KBUx, Package_DFN_QFN:QFN-32-1EP_5x5mm_P0.5mm_EP3.45x3.45mm, symbol MCU_ST_STM32L4:STM32L431KBUx
- added R22, R23, R24, R25: 100K, Capacitor_SMD:C_0402_1005Metric, symbol Device:R_Small
- added U9: STM32L432KBUx, Package_DFN_QFN:QFN-32-1EP_5x5mm_P0.5mm_EP3.45x3.45mm, symbol MCU_ST_STM32L4:STM32L432KBUx
Connections:
- net GND: now also U9.16 (VSS), U9.32 (VSS), U9.33 (VSS)
- net I2C_SCL: now also R20.1, U9.19 (PA9); no longer R20.2
- net I2C_SDA: now also R19.1, U9.20 (PA10); no longer R19.2
- net P3V3: now also R19.2, R20.2, R22.2, R23.2, R24.2, R25.2, U9.1 (VDD), U9.17 (VDD), U9.5 (VDDA); no longer R19.1, R20.1
- net SWCLK: now also U9.24 (PA14)
- net SWDIO: now also U9.23 (PA13)
- net ~{nRST}: now also U9.4 (NRST)
- net at R17.1: now also U9.31 (PH3)
- net at SW1.6: now also R23.1, U9.26 (PB3)
- net at D3.2 (A): now also U9.12 (PA6)
- net at SW1.7: now also R24.1, U9.15 (PB1)
- net at SW1.5: now also R22.1, U9.27 (PB4)
- net at D2.2 (A): now also U9.13 (PA7)
- net at SW1.8: now also R25.1, U9.14 (PB0)
- net at R18.1, U2.5 (WP): now also U9.6 (PA0)
- new net CAN_RX: U9.21 (PA11)
- new net CAN_STANDBY: U9.18 (PA8)
- new net CAN_TX: U9.22 (PA12)
- new net UART_RX: U9.9 (PA3)
- new net UART_TX: U9.8 (PA2)
- no-connect marks 4 -> 11
Other:
- note added: "4-bit Sensor Address"
- note removed: "Sensor Address"
- moved on the sheet: D2, D3, R1, R19, R2, R20

Commit message: mostly done with sensor module
Connections:
- net at R25.1, SW1.8: now also U9.29 (PB6); no longer U9.14 (PB0)
- net at R24.1, SW1.7: now also U9.28 (PB5); no longer U9.15 (PB1)
- net at R23.1, SW1.6: now also U9.27 (PB4); no longer U9.26 (PB3)
- net at R22.1, SW1.5: now also U9.26 (PB3); no longer U9.27 (PB4)
Changed lines of the file:
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@@
-	)
-	(junction
-		(at 83.82 105.41)
-		(diameter 0)
-		(color 0 0 0 0)
 	)
 	(junction
@@
 	)
 	(junction
+		(at 119.38 35.56)
+		(diameter 0)
+		(color 0 0 0 0)
+	)
+	(junction
+		(at 203.2 119.38)
+		(diameter 0)
+		(color 0 0 0 0)
+	)
+	(junction
+		(at 156.21 87.63)
+		(diameter 0)
+		(color 0 0 0 0)
+	)
+	(junction
+		(at 109.22 55.88)
+		(diameter 0)
+		(color 0 0 0 0)
+	)
+	(junction
+		(at 74.93 121.92)
+		(diameter 0)
+		(color 0 0 0 0)
+	)
+	(junction
+		(at 91.44 64.77)
+		(diameter 0)
+		(color 0 0 0 0)
+	)
+	(junction
 		(at 92.71 102.87)
 		(diameter 0)
@@
 	)
 	(junction
-		(at 119.38 35.56)
-		(diameter 0)
-		(color 0 0 0 0)
-	)
-	(junction
-		(at 203.2 119.38)
-		(diameter 0)
-		(color 0 0 0 0)
-	)
-	(junction
-		(at 156.21 87.63)
-		(diameter 0)
-		(color 0 0 0 0)
-	)
-	(junction
-		(at 109.22 55.88)
-		(diameter 0)
-		(color 0 0 0 0)
-	)
-	(junction
-		(at 74.93 121.92)
-		(diameter 0)
-		(color 0 0 0 0)
-	)
-	(junction
-		(at 91.44 64.77)
+		(at 74.93 107.95)
 		(diameter 0)
 		(color 0 0 0 0)
@@
 	)
 	(junction
+		(at 125.73 35.56)
+		(diameter 0)
+		(color 0 0 0 0)
+	)
+	(junction
+		(at 123.19 55.88)
+		(diameter 0)
+		(color 0 0 0 0)
+	)
+	(junction
+		(at 134.62 55.88)
+		(diameter 0)
+		(color 0 0 0 0)
+	)
+	(junction
+		(at 134.62 35.56)
+		(diameter 0)
+		(color 0 0 0 0)
+	)
+	(junction
+		(at 125.73 55.88)
+		(diameter 0)
+		(color 0 0 0 0)
+	)
+	(junction
+		(at 127 55.88)
+		(diameter 0)
+		(color 0 0 0 0)
+	)
+	(junction
 		(at 101.6 100.33)
 		(diameter 0)
@@
 	)
 	(junction
-		(at 125.73 35.56)
-		(diameter 0)
-		(color 0 0 0 0)
-	)
-	(junction
-		(at 123.19 55.88)
-		(diameter 0)
-		(color 0 0 0 0)
-	)
-	(junction
-		(at 134.62 55.88)
-		(diameter 0)
-		(color 0 0 0 0)
-	)
-	(junction
-		(at 134.62 35.56)
-		(diameter 0)
-		(color 0 0 0 0)
-	)
-	(junction
-		(at 74.93 107.95)
-		(diameter 0)
-		(color 0 0 0 0)
-	)
-	(junction
-		(at 125.73 55.88)
-		(diameter 0)
-		(color 0 0 0 0)
-	)
-	(junction
-		(at 127 55.88)
+		(at 80.01 105.41)
 		(diameter 0)
 		(color 0 0 0 0)
@@
 	)
 	(no_connect
-		(at 113.03 95.25)
+		(at 113.03 77.47)
 	)
 	(no_connect
-		(at 113.03 77.47)
-	)
-	(no_connect
-		(at 113.03 92.71)
+		(at 113.03 85.09)
 	)
 	(no_connect
@@
 		(at 64.77 59.69)
 	)
-	(wire
-		(pts
-			(xy 113.03 90.17) (xy 74.93 90.17)
-		)
-		(stroke
-			(width 0)
-			(type default)
-		)
+	(no_connect
+		(at 113.03 82.55)
 	)
 	(wire
@@
 	(wire
 		(pts
-			(xy 92.71 85.09) (xy 92.71 102.87)
-		)
-		(stroke
-			(width 0)
-			(type default)
-		)
-	)
-	(wire
-		(pts
 			(xy 134.62 55.88) (xy 134.62 49.53)
 		)
@@
 	(wire
 		(pts
+			(xy 74.93 87.63) (xy 74.93 107.95)
+		)
+		(stroke
+			(width 0)
+			(type default)
+		)
+	)
+	(wire
+		(pts
 			(xy 127 55.88) (xy 128.27 55.88)
 		)
@@
 	(wire
 		(pts
+			(xy 80.01 90.17) (xy 80.01 105.41)
+		)
+		(stroke
+			(width 0)
+			(type default)
+		)
+	)
+	(wire
+		(pts
 			(xy 203.2 119.38) (xy 194.31 119.38)
 		)
@@
 	(wire
 		(pts
-			(xy 113.03 87.63) (xy 83.82 87.63)
-		)
-		(stroke
-			(width 0)
-			(type default)
-		)
-	)
-	(wire
-		(pts
-			(xy 113.03 85.09) (xy 92.71 85.09)
-		)
-		(stroke
-			(width 0)
-			(type default)
-		)
-	)
-	(wire
-		(pts
 			(xy 83.82 121.92) (xy 83.82 116.84)
 		)
@@
 	(wire
 		(pts
+			(xy 92.71 92.71) (xy 92.71 102.87)
+		)
+		(stroke
+			(width 0)
+			(type default)
+		)
+	)
+	(wire
+		(pts
 			(xy 119.38 35.56) (xy 119.38 44.45)
 		)
@@
 	(wire
 		(pts
+			(xy 113.03 95.25) (xy 101.6 95.25)
+		)
+		(stroke
+			(width 0)
+			(type default)
+		)
+	)
+	(wire
+		(pts
 			(xy 194.31 109.22) (xy 194.31 111.76)
 		)
@@
 	(wire
 		(pts
+			(xy 113.03 92.71) (xy 92.71 92.71)
+		)
+		(stroke
+			(width 0)
+			(type default)
+		)
+	)
+	(wire
+		(pts
 			(xy 125.73 35.56) (xy 127 35.56)
 		)
@@
 	(wire
 		(pts
+			(xy 113.03 87.63) (xy 74.93 87.63)
+		)
+		(stroke
+			(width 0)
+			(type default)
+		)
+	)
+	(wire
+		(pts
 			(xy 125.73 55.88) (xy 127 55.88)
 		)
@@
 	(wire
 		(pts
-			(xy 101.6 82.55) (xy 101.6 100.33)
-		)
-		(stroke
-			(width 0)
-			(type default)
-		)
-	)
-	(wire
-		(pts
 			(xy 55.88 107.95) (xy 53.34 107.95)
 		)
@@
 	(wire
 		(pts
-			(xy 113.03 82.55) (xy 101.6 82.55)
-		)
-		(stroke
-			(width 0)
-			(type default)
-		)
-	)
-	(wire
-		(pts
 			(xy 127 35.56) (xy 134.62 35.56)
 		)
@@
 	(wire
 		(pts
-			(xy 71.12 105.41) (xy 83.82 105.41)
+			(xy 71.12 105.41) (xy 80.01 105.41)
 		)
 		(stroke
@@
 	(wire
 		(pts
-			(xy 74.93 90.17) (xy 74.93 107.95)
-		)
-		(stroke
-			(width 0)
-			(type default)
-		)
-	)
-	(wire
-		(pts
 			(xy 101.6 100.33) (xy 101.6 111.76)
 		)
@@
 	(wire
 		(pts
-			(xy 83.82 87.63) (xy 83.82 105.41)
-		)
-		(stroke
-			(width 0)
-			(type default)
-		)
-	)
-	(wire
-		(pts
 			(xy 119.38 35.56) (xy 109.22 35.56)
 		)
@@
 	(wire
 		(pts
+			(xy 113.03 90.17) (xy 80.01 90.17)
+		)
+		(stroke
+			(width 0)
+			(type default)
+		)
+	)
+	(wire
+		(pts
 			(xy 71.12 100.33) (xy 101.6 100.33)
 		)
@@
 	(wire
 		(pts
+			(xy 80.01 105.41) (xy 83.82 105.41)
+		)
+		(stroke
+			(width 0)
+			(type default)
+		)
+	)
+	(wire
+		(pts
 			(xy 194.31 82.55) (xy 194.31 104.14)
 		)
@@
 		)
 		(stroke
+			(width 0)
+			(type default)
+		)
+	)
+	(wire
+		(pts
+			(xy 101.6 95.25) (xy 101.6 100.33)
+		)
+		(stroke
