File: co2_hub/cell.kicad_sch (KiCad schematic)
At the start: 12 parts, among them J2 Conn_ARM_SWD_TagConnect_TC203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, U3 NRF9151-LACA-R7

Commit message: mostly done with sensor module
Parts:
- removed R1: 10K, symbol Device:R_Small
- C16: value 100nF -> 0.1uF
- U3: LCSC (none) -> C42236596
Connections:
- net ENABLE: now reaches U3.10 (ENABLE)
Changed lines of the file:
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@@
-	)
-	(junction
-		(at 166.37 54.61)
-		(diameter 0)
-		(color 0 0 0 0)
 	)
 	(junction
@@
 	(wire
 		(pts
+			(xy 110.49 67.31) (xy 111.76 67.31)
+		)
+		(stroke
+			(width 0)
+			(type default)
+		)
+	)
+	(wire
+		(pts
 			(xy 189.23 43.18) (xy 212.09 43.18)
 		)
@@
 	(wire
 		(pts
-			(xy 166.37 40.64) (xy 166.37 54.61)
-		)
-		(stroke
-			(width 0)
-			(type default)
-		)
-	)
-	(wire
-		(pts
 			(xy 167.64 35.56) (xy 172.72 35.56)
 		)
@@
 	(wire
 		(pts
-			(xy 104.14 53.34) (xy 104.14 40.64)
-		)
-		(stroke
-			(width 0)
-			(type default)
-		)
-	)
-	(wire
-		(pts
-			(xy 104.14 67.31) (xy 111.76 67.31)
-		)
-		(stroke
-			(width 0)
-			(type default)
-		)
-	)
-	(wire
-		(pts
 			(xy 162.56 52.07) (xy 172.72 52.07)
 		)
@@
 	(wire
 		(pts
-			(xy 162.56 54.61) (xy 166.37 54.61)
-		)
-		(stroke
-			(width 0)
-			(type default)
-		)
-	)
-	(wire
-		(pts
 			(xy 172.72 22.86) (xy 172.72 29.21)
 		)
@@
 	(wire
 		(pts
-			(xy 104.14 58.42) (xy 104.14 67.31)
-		)
-		(stroke
-			(width 0)
-			(type default)
-		)
-	)
-	(wire
-		(pts
 			(xy 180.34 22.86) (xy 180.34 29.21)
 		)
@@
 	(wire
 		(pts
-			(xy 104.14 40.64) (xy 166.37 40.64)
-		)
-		(stroke
-			(width 0)
-			(type default)
-		)
-	)
-	(wire
-		(pts
 			(xy 153.67 35.56) (xy 162.56 35.56)
 		)
@@
 	(wire
 		(pts
-			(xy 166.37 54.61) (xy 180.34 54.61)
+			(xy 162.56 54.61) (xy 180.34 54.61)
 		)
 		(stroke
@@
 			)
 			(justify left)
+		)
+	)
+	(hierarchical_label "ENABLE"
+		(shape input)
+		(at 110.49 67.31 180)
+		(effects
+			(font
+				(size 1.27 1.27)
+			)
+			(justify right)
 		)
 	)
@@
 				(path "/032ed60e-c83d-45fe-8a79-75f890542253/55ec85ad-7e05-4c9c-aa3d-f086fc8d1c1d"
 					(reference "C2")
-					(unit 1)
-				)
-			)
-		)
-	)
-	(symbol
-		(lib_id "Device:R_Small")
-		(at 104.14 55.88 0)
-		(mirror x)
-		(unit 1)
-		(body_style 1)
-		(exclude_from_sim no)
-		(in_bom yes)
-		(on_board yes)
-		(in_pos_files yes)
-		(dnp no)
-		(fields_autoplaced yes)
-		(property "Reference" "R1"
-			(at 101.6 54.6099 0)
-			(show_name no)
-			(do_not_autoplace no)
-			(effects
-				(font
-					(size 1.016 1.016)
-				)
-				(justify right)
-			)
-		)
-		(property "Value" "10K"
-			(at 101.6 57.1499 0)
-			(show_name no)
-			(do_not_autoplace no)
-			(effects
-				(font
-					(size 1.27 1.27)
-				)
-				(justify right)
-			)
-		)
-		(property "Footprint" ""
-			(at 104.14 55.88 0)
-			(hide yes)
-			(show_name no)
-			(do_not_autoplace no)
-			(effects
-				(font
-					(size 1.27 1.27)
-				)
-			)
-		)
-		(property "Datasheet" ""
-			(at 104.14 55.88 0)
-			(hide yes)
-			(show_name no)
-			(do_not_autoplace no)
-			(effects
-				(font
-					(size 1.27 1.27)
-				)
-			)
-		)
-		(property "Description" "Resistor, small symbol"
-			(at 104.14 55.88 0)
-			(hide yes)
-			(show_name no)
-			(do_not_autoplace no)
-			(effects
-				(font
-					(size 1.27 1.27)
-				)
-			)
-		)
-		(pin "2"
-		)
-		(pin "1"
-		)
-		(instances
-			(project "co2_hub"
-				(path "/032ed60e-c83d-45fe-8a79-75f890542253/55ec85ad-7e05-4c9c-aa3d-f086fc8d1c1d"
-					(reference "R1")
 					(unit 1)
 				)
@@
 			)
 		)
+		(property "LCSC" "C42236596"
+			(at 137.16 95.25 0)
+			(hide yes)
+			(show_name no)
+			(do_not_autoplace no)
+			(effects
+				(font
+					(size 1.27 1.27)
+				)
+			)
+		)
 		(pin "38"
 		)
@@
 			)
 		)
-		(property "Value" "100nF"
+		(property "Value" "0.1uF"
 			(at 161.29 37.338 90)
 			(show_name no)

Commit message: (mostly) finalized sensing units + progress on surface hub
Parts:
- removed C2, C5: 1uF, symbol Device:C_Small
- removed C6: 10uF, symbol Device:C_Small
- added C24, C28: 100nF, Capacitor_SMD:C_0402_1005Metric, symbol Device:C_Small
- added C25, C26, C27: 20pF, Capacitor_SMD:C_0402_1005Metric, symbol Device:C_Small
- added C29, C30: 1uF, Capacitor_SMD:C_0603_1608Metric, symbol Device:C_Small
- added J3: SIM_Card_Shielded, Connector_JAE:JAE_SIM_Card_SF72S006, symbol Connector:SIM_Card_Shielded
- added J4: Conn_Coaxial, symbol Connector:Conn_Coaxial
- added R22: 10K, Resistor_SMD:R_0402_1005Metric, symbol Device:R_Small
- C1: footprint (none) -> Capacitor_SMD:C_1206_3216Metric; LCSC (none) -> C96123
- C15: footprint (none) -> Capacitor_SMD:C_0603_1608Metric; LCSC (none) -> C19666
- C16: value 0.1uF -> 4.7uF; footprint (none) -> Capacitor_SMD:C_0603_1608Metric; LCSC (none) -> C19666
- C17: value 4.7uF -> 10uF; footprint (none) -> Capacitor_SMD:C_0805_2012Metric; LCSC (none) -> C15850
- C23: value 0.1uF -> 100nF; footprint (none) -> Capacitor_SMD:C_0402_1005Metric; LCSC (none) -> C1525
- FB1: footprint (none) -> Capacitor_SMD:C_0603_1608Metric; LCSC (none) -> C361652
Connections:
- net SWCLK is gone; now on net SW_CLK: J2.4 (SWCLK)
- net SWDIO is gone; now on net SW_DIO: J2.2 (SWDIO)
- net GND: now also C15.1, C24.1, C25.1, C26.1, C27.2, C28.1, C29.2, C30.2, J3.5 (GND), J3.SH, J4.2 (Ext); no longer C15.2
- net P3V3: now also C15.2, C28.2; no longer C15.1, C16.1
- net P5V0: now also C29.1, C30.1, R22.1
- net at FB1.1, U3.14 (VDD): now also C17.1
- net at U3.24 (DEC0): now also C16.1; no longer C17.1
- net SIM_RST: now reaches U3.16 (SIM_RST)
- net SIM_RST: now also C26.2, J3.2 (RST)
- net SIM_IO: now reaches U3.17 (SIM_IO)
- net SIM_IO: now also C27.1, J3.7 (I/O)
- net SIM_CLK: now reaches U3.18 (SIM_CLK)
- net SIM_CLK: now also C25.2, J3.3 (CLK)
- net SIM_P1V8: now reaches U3.19 (SIM_1V8)
- net SIM_P1V8: now also C24.2, J3.1 (VCC)
- net SW_CLK: now reaches U3.3 (SWDCLK)
- net at U3.35 (ANT): now also J4.1 (In)
- net SW_DIO: now reaches U3.4 (SWDIO)
- net ~{nCELL_RI}: now reaches U3.49 (P0.30)
- net CELL_DTR: now reaches U3.50 (P0.31)
- net CELL_TX: now reaches U3.58 (P0.02)
- net CELL_RX: now reaches U3.59 (P0.03)
- net CELL_RTS: now reaches U3.63 (P0.06)
- net CELL_CTS: now reaches U3.64 (P0.07)
- net ENABLE: no longer names the net of U3.10 (ENABLE)
- net ENABLE: now also R22.2
- no-connect marks 2 -> 7
Other:
- note added: "The 20pF caps are for ESD protection"
- note removed: "These caps are kinda whack but the hardware sheet says so lol"
- moved on the sheet: C1, FB1, J2, U3A
