File: co2_hub/mcu.kicad_sch (KiCad schematic)
At the start: 14 parts, among them J1 Conn_ARM_SWD_TagConnect_TC203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, U1 STM32L433RCTx, U2 CBLW 24C02

Commit message: (mostly) finalized sensing units + progress on surface hub
Parts:
- added C2, C5: 13pF, Capacitor_SMD:C_0402_1005Metric, symbol Device:C_Small
- added Y1: 25MHz, Crystal:Crystal_SMD_3225-4Pin_3.2x2.5mm, symbol Device:Crystal_Small
Connections:
- net GND: now also C2.1, C5.1
- net LPUART1_CTS: now reaches U1.22 (PA6)
- net LPUART1_RTS: now reaches U1.27 (PB1)
- net at U1.5 (PH0): now also C2.2, Y1.2
- net UART1_TX: now reaches U1.58 (PB6)
- net UART1_RX: now reaches U1.59 (PB7)
- net at U1.6 (PH1): now also C5.2, Y1.1
- net LPUART1_RX: now reaches U1.8 (PC0)
- net LPUART1_TX: now reaches U1.9 (PC1)
- no-connect marks 5 -> 3
Other:
- moved on the sheet: J1, R17
