File: co2_hub/solar.kicad_sch (KiCad schematic)
At the start: 0 parts

Commit message: progress on solar charging + misc
Parts:
- added C31, C32: 10uF, Capacitor_SMD:C_0805_2012Metric, symbol Device:C_Small
- added C6: 1uF, symbol Device:C_Small
- added D1, D2, D3, D5: D_Schottky_Small, Package_SO:MSOP-12-1EP_3x4.039mm_P0.65mm_EP1.651x2.845mm, symbol Device:D_Schottky_Small
- added D4: Zener 6.2V, Diode_SMD:D_SOD-123, symbol Device:D_Zener_Small
- added L3: 10uH, symbol Device:L_Small
- added R1: 0.05, Resistor_SMD:R_1206_3216Metric, symbol Device:R_Small
- added U9: LT3652IMSE, Package_SO:MSOP-12-1EP_3x4.039mm_P0.65mm_EP1.651x2.845mm, symbol Battery_Management:LT3652IMSE
Connections:
- new net: D3.2 (A), D4.2 (A)
- new net: C6.2, D3.1 (K), U9.11 (BOOST)
- new net: C6.1, D5.1 (K), L3.1, U9.12 (SW)
- new net: C31.2, D1.1 (K), U9.1 (V_{IN})
- new net BAT: C32.1, D2.2 (A), D4.1 (K), R1.2, U9.9 (BAT)
- new net GND: C31.1, C32.2, D5.2 (A), U9.13 (GND)
- new net SENSE: L3.2, R1.1, U9.10 (SENSE)
- new net Vbus: D2.1 (K)
- new net Vsolar: D1.2 (A)
Other:
- note added: "TODO: BMS will go here"
